File: electronics/Sensor_V1.0/Sensor_V1.0.kicad_pcb (KiCad board)
At the start: 2 copper layers, 45.9 x 25.6 mm, 55 parts, among them J1 nuclone_small_left, J2 nuclone_small_right, J5 DevBoardUartInput, Q1 BC846, U1 PPG_sensor, U2 reference_sot23-3, U3 MCP6541

Commit message: beautified position a bit (ordering of capacitor to be incrementing
Parts:
- moved C7 1.90 mm to (79.5, 86.3)
- moved C8 1.90 mm to (81.4, 86.3)
Changed lines of the file:
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@@
   )
   (module SquantorRcl:C_0805+0603 (layer B.Cu)
-    (at 79.5 86.3 270)
+    (at 81.4 86.3 270)
     (descr "Capacitor SMD 0805 and 0603 pad sizes, reflow soldering, based on AVX dimensions")
     (tags "capacitor 0805 0603 mixed")
@@
   )
   (module SquantorRcl:C_0805+0603 (layer B.Cu)
-    (at 81.4 86.3 270)
+    (at 79.5 86.3 270)
     (descr "Capacitor SMD 0805 and 0603 pad sizes, reflow soldering, based on AVX dimensions")
     (tags "capacitor 0805 0603 mixed")

Commit message: updated versionnumber
Parts:
- N2: value 20200810 -> 20200811
Changed lines of the file:
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@@
       (effects (font (size 1 1) (thickness 0.15)))
     )
-    (fp_text value 20200810 (at 0.8 -0.1) (layer F.SilkS)
+    (fp_text value 20200811 (at 0.8 -0.1) (layer F.SilkS)
       (effects (font (size 0.8 0.8) (thickness 0.15)))
     )
