File: electronics/Sensor_V1.2/Sensor_V1.2.kicad_pcb (KiCad board)
At the start: 2 copper layers, 45.9 x 25.6 mm, 35 parts, among them J1 nuclone_small_left, J2 nuclone_small_right, J3 Proto_1pin, J5 DevBoardUartInput, Q1 DMG1012, U1 PPG_sensor

Commit message: added notes field, updated versionnumber
Parts:
- added N4: notes:, SquantorLabels:Label_Note_medium, F.Cu at (89.8, 97.0)
- N2: value 20210215 -> 20210217
- R8: value 100K -> 4.7K

Commit message: added plotting outputs
Other:
- rule pad_to_mask_clearance: 0.1 -> 0
